File: Hardware/SparkFun_Qwiic_Distance - VL53L4CD.sch (EAGLE design)
At the start: 27 parts, among them J2 QWIIC_RIGHT_ANGLE, J4 QWIIC_RIGHT_ANGLE, U1 VL53L4CX

Commit message: Updates Distance Sensor Part name
Parts:
- U1: value VL53L4CX -> VL53L4CD; device DISTANCE:VL53L4CX -> DISTANCE:VL53L4CD
Changed lines of the file:
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@@
 <?xml version="1.0" encoding="utf-8"?>
 <!DOCTYPE eagle SYSTEM "eagle.dtd">
-<eagle version="9.6.2">
+<eagle version="9.5.1">
 <drawing>
 <settings>
@@
 <part name="GND3" library="SparkFun-PowerSymbols" deviceset="GND" device=""/>
 <part name="FRAME1" library="SparkFun-Aesthetics" deviceset="FRAME-LETTER" device=""/>
-<part name="U1" library="DISTANCE" deviceset="VL53L4CX" device=""/>
+<part name="U1" library="DISTANCE" deviceset="VL53L4CD" device=""/>
 <part name="J7" library="SparkFun-Connectors" deviceset="CONN_06" device="NO_SILK_NO_POP"/>
 <part name="SUPPLY11" library="SparkFun-PowerSymbols" deviceset="3.3V" device=""/>
